File: Modules/hackpad-mine-slider/hackpad-mine-slider.kicad_pcb (KiCad board)
At the start: 4 copper layers, 81.6 x 35.5 mm, 52 parts, among them J1 UPDI_Common, J2 Right_Connector, J3 Bottom_Connector, J4 Left_Connector, J5 Top_Connector, Q1 PMOS, SW4 SW_SPDT, U1 ATtiny1616-S, U2 TMUX4052, U3 ATtiny414-SS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

Commit message: updated pcb silkscreen for prettification
Other:
- board text removed: "cool image here :3"
Changed lines of the file:
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@@
 		(tags "VSSOP SO JEDEC-MO-187-CA TI-DCU0008A")
 		(property "Reference" "U4"
-			(at 0 -1.95 90)
+			(at 0 2.3 90)
 			(layer "F.SilkS")
 			(effects
@@
 		(tags "Diode Mini-MELF (SOD-80) Handsoldering")
 		(property "Reference" "D5"
-			(at 0 -2 0)
+			(at 0 2 0)
 			(layer "F.SilkS")
 			(effects
@@
 		(tags "capacitor handsolder")
 		(property "Reference" "C8"
-			(at 2.3 0 180)
+			(at -2.7 0 180)
 			(layer "F.SilkS")
 			(effects
@@
 		(tags "capacitor handsolder")
 		(property "Reference" "C6"
-			(at 2.2375 -1.95 0)
+			(at -2.6625 0.05 0)
 			(layer "F.SilkS")
 			(effects
@@
 		(tags "VSSOP SO JEDEC-MO-187-AA TI-DGK0008A")
 		(property "Reference" "U8"
-			(at 0 2.45 0)
+			(at 0 -2.525 0)
 			(layer "B.SilkS")
 			(effects
@@
 		(tags "VSSOP SO JEDEC-MO-187-CA TI-DCU0008A")
 		(property "Reference" "U7"
-			(at 0 1.95 90)
+			(at 0 -2.18 90)
 			(layer "B.SilkS")
 			(effects
@@
 		(tags "SOT-23 AO3401A")
 		(property "Reference" "Q1"
-			(at 1.45 1.58 0)
+			(at 1.65 1.9625 0)
 			(layer "B.SilkS")
 			(effects
@@
 		(tags "capacitor handsolder")
 		(property "Reference" "C3"
-			(at -2.8 0 0)
+			(at 3.2 0 0)
 			(layer "B.SilkS")
 			(effects
@@
 		(tags "resistor handsolder")
 		(property "Reference" "R1"
-			(at 3.2 0.1 90)
+			(at 0 -2.2 90)
 			(layer "B.SilkS")
 			(effects
@@
 		)
 	)
-	(gr_text "cool image here :3"
-		(at 219.685 77.398752 -0)
-		(layer "B.SilkS")
-		(effects
-			(font
-				(size 1 1)
-				(thickness 0.2)
-				(bold yes)
-			)
-			(justify left bottom mirror)
-		)
-	)
